File: Layout/Avalon16.sch (EAGLE design)
At the start: 229 parts, among them IC1 PTH12040WAH, IC10 A3255Q48, IC11 A3255Q48, IC12 A3255Q48, IC13 A3255Q48, IC14 A3255Q48, IC15 A3255Q48, IC16 A3255Q48, IC17 A3255Q48, IC19 A3255Q48, IC2 NB3L553DG, IC20 A3255Q48, IC3 LM2576S-3.3, IC4 PIC16LF1459, IC5 74HC02D, IC6 A3255Q48, IC7 A3255Q48, IC8 A3255Q48, IC9 A3255Q48, Q1 7W-25-000MBB-T, Q2 IRFML8244TRPBF, X1 Molex 45558-0003, X2 ISP, X3 Molex 22-04-1031, X4 Würth 65100516121 / TE 173403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

Commit message: add level translator
Parts:
- added C125: 0.1µ, rcl:C-EUC0805
- added C126: 1µ, rcl:C-EUC0805
- added U$1: GTL2003, GTL2003:GTL2003
Connections:
- new net CONFIG1_1V8_N: IC6.CONFIG_NI@2, U$1.S2
- new net CONFIG1_1V8_P: IC6.CONFIG_PI@1, U$1.S1
- new net CONFIG2_1V8_N: IC11.CONFIG_NI@2, U$1.S4
- new net CONFIG2_1V8_P: IC11.CONFIG_PI@1, U$1.S3
- new net N$11: U$1.D7
- new net N$12: U$1.D8
- new net N$13: U$1.S7
- new net N$14: U$1.S8
- new net REPORT_1V8_N: U$1.S6
- new net REPORT_1V8_P: U$1.S5
- new net V+: C125.1, U$1.SREF
- net +3V3: now also C126.1, U$1.DREF, U$1.GREF
- net CONFIG1_N: now also U$1.D2; no longer IC6.CONFIG_NI@2
- net CONFIG1_P: now also U$1.D1; no longer IC6.CONFIG_PI@1
- net CONFIG2_N: now also U$1.D4; no longer IC11.CONFIG_NI@2
- net CONFIG2_P: now also U$1.D3; no longer IC11.CONFIG_PI@1
- net GND: now also C125.2, C126.2, U$1.GND
- net REPORT_N: now also U$1.D6
- net REPORT_P: now also U$1.D5
Other:
- note added: "Avalon Gen3 Support"
- note removed: "Notes"
